Commit message: feat: add fine picker urdf

File: descriptions/simple_picker/urdf/picker.urdf (robot description, URDF)
Before this commit: robot picker, 5 links, 4 joints
Joints:
- joint base_link_to_link2: limit lower=0 upper=1.3 effort=1000.0 velocity=0.5 -> lower=0 upper=1.3 effort=1000.0 velocity=1.2
- joint link2_to_link3_1: axis -0.9999955995433731 0.002966618003841546 -0.000008456311998861208 -> -1 0 0; limit lower=0 upper=0.8 effort=1000.0 velocity=0.5 -> lower=0 upper=0.7 effort=1000.0 velocity=1.2; origin xyz=0.5 0.08 0 rpy=0 0 0 -> xyz=0.40 0.08 0 rpy=0 0 0
- joint link3_1_to_link4_1: limit lower=-0.7 upper=0 effort=1000.0 velocity=0.5 -> lower=-0.9 upper=0 effort=1000.0 velocity=1.2
